File: oresat-backplane.sch (EAGLE design)
At the start: 10 parts, among them J1 SFM-120-X1-XXX-D, J2 SFM-120-X1-XXX-D

Commit message: Beginnings of the 20 slots, with connectors! Almost Joe Approved, waiting for better DXF.
Parts:
- added CF10, CF11, CF13, CF14, CF15, CF17, CF18, CF19, CF21, CF22, CF23, CF25, CF26, CF27, CF9: ORESAT-BACKPLANE-TO-UT-047, J-Cinch-MMCX-135-3701-211-to-UT-047:ORESAT-BACKPLANE-TO-UT-047
- added CF12, CF16, CF20, CF24, CF28: SFM-110-X1-XXX-D-LC, J-Samtec-SFM-110-X1-XXX-D-LC:SFM-110-X1-XXX-D-LC
- added J3, J4, J5, J6, J7: SFM-120-X1-XXX-D, J-Samtec-SFM-120-X1-XXX-D:SFM-120-X1-XXX-D
Connections:
- net !SHUTDOWN: now also J3.7, J3.8, J4.7, J4.8, J5.7, J5.8, J6.7, J6.8, J7.7, J7.8
- net CAN_H: now also J3.3, J3.4, J4.3, J4.4, J5.3, J5.4, J6.3, J6.4, J7.3, J7.4
- net CAN_L: now also J3.1, J3.2, J4.1, J4.2, J5.1, J5.2, J6.1, J6.2, J7.1, J7.2
- net GND: now also CF10.SHIELD, CF10.SHIELD1, CF10.SHIELD2, CF10.SHIELD3, CF11.SHIELD, CF11.SHIELD1, CF11.SHIELD2, CF11.SHIELD3, CF12.LC1, CF12.LC2, CF13.SHIELD, CF13.SHIELD1, CF13.SHIELD2, CF13.SHIELD3, CF14.SHIELD, CF14.SHIELD1, CF14.SHIELD2, CF14.SHIELD3, CF15.SHIELD, CF15.SHIELD1, CF15.SHIELD2, CF15.SHIELD3, CF16.LC1, CF16.LC2, CF17.SHIELD, CF17.SHIELD1, CF17.SHIELD2, CF17.SHIELD3, CF18.SHIELD, CF18.SHIELD1, CF18.SHIELD2, CF18.SHIELD3, CF19.SHIELD, CF19.SHIELD1, CF19.SHIELD2, CF19.SHIELD3, CF20.LC1, CF20.LC2, CF21.SHIELD, CF21.SHIELD1, CF21.SHIELD2, CF21.SHIELD3, CF22.SHIELD, CF22.SHIELD1, CF22.SHIELD2, CF22.SHIELD3, CF23.SHIELD, CF23.SHIELD1, CF23.SHIELD2, CF23.SHIELD3, CF24.LC1, CF24.LC2, CF25.SHIELD, CF25.SHIELD1, CF25.SHIELD2, CF25.SHIELD3, CF26.SHIELD, CF26.SHIELD1, CF26.SHIELD2, CF26.SHIELD3, CF27.SHIELD, CF27.SHIELD1, CF27.SHIELD2, CF27.SHIELD3, CF28.LC1, CF28.LC2, CF4.SHIELD1, CF4.SHIELD2, CF4.SHIELD3, CF5.SHIELD1, CF5.SHIELD2, CF5.SHIELD3, CF6.SHIELD1, CF6.SHIELD2, CF6.SHIELD3, CF9.SHIELD, CF9.SHIELD1, CF9.SHIELD2, CF9.SHIELD3, J3.10, J3.11, J3.12, J3.5, J3.6, J3.9, J3.LC1, J3.LC2, J4.10, J4.11, J4.12, J4.5, J4.6, J4.9, J4.LC1, J4.LC2, J5.10, J5.11, J5.12, J5.5, J5.6, J5.9, J5.LC1, J5.LC2, J6.10, J6.11, J6.12, J6.5, J6.6, J6.9, J6.LC1, J6.LC2, J7.10, J7.11, J7.12, J7.5, J7.6, J7.9, J7.LC1, J7.LC2
- net VBUS: now also J3.13, J3.14, J3.15, J3.16, J4.13, J4.14, J4.15, J4.16, J5.13, J5.14, J5.15, J5.16, J6.13, J6.14, J6.15, J6.16, J7.13, J7.14, J7.15, J7.16

Commit message: OMG we have a backplane. Note that the MMCX connectors are probably incorrectly placed because we're going to switch to some different connector that's more SMT-y for Oliver because he's an RF racist.
Parts:
- added CF29, CF30, CF31, CF33, CF34, CF35, CF37, CF38, CF39, CF41, CF42, CF43, CF45, CF46, CF47, CF49, CF50, CF51, CF53, CF54, CF55, CF57, CF58, CF59, CF61, CF62, CF63, CF65, CF66, CF67, CF69, CF70, CF71, CF73, CF74, CF75, CF77, CF78, CF79: ORESAT-BACKPLANE-TO-UT-047, J-Cinch-MMCX-135-3701-211-to-UT-047:ORESAT-BACKPLANE-TO-UT-047
- added CF32, CF36, CF40, CF44, CF48, CF52, CF56, CF60, CF64, CF68, CF72, CF76, CF80: SFM-110-X1-XXX-D-LC, J-Samtec-SFM-110-X1-XXX-D-LC:SFM-110-X1-XXX-D-LC
- added J10, J11, J12, J13, J15, J16, J17, J18, J19, J8, J9: SFM-120-X1-XXX-D, J-Samtec-SFM-120-X1-XXX-D:SFM-120-X1-XXX-D
- renumbered J1 to J14
Connections:
- net !SHUTDOWN: now also J10.7, J10.8, J11.7, J11.8, J12.7, J12.8, J13.7, J13.8, J15.7, J15.8, J16.7, J16.8, J17.7, J17.8, J18.7, J18.8, J19.7, J19.8, J8.7, J8.8, J9.7, J9.8
- net CAN_H: now also J10.3, J10.4, J11.3, J11.4, J12.3, J12.4, J13.3, J13.4, J15.3, J15.4, J16.3, J16.4, J17.3, J17.4, J18.3, J18.4, J19.3, J19.4, J8.3, J8.4, J9.3, J9.4
- net CAN_L: now also J10.1, J10.2, J11.1, J11.2, J12.1, J12.2, J13.1, J13.2, J15.1, J15.2, J16.1, J16.2, J17.1, J17.2, J18.1, J18.2, J19.1, J19.2, J8.1, J8.2, J9.1, J9.2
- net GND: now also CF29.SHIELD, CF29.SHIELD1, CF29.SHIELD2, CF29.SHIELD3, CF30.SHIELD, CF30.SHIELD1, CF30.SHIELD2, CF30.SHIELD3, CF31.SHIELD, CF31.SHIELD1, CF31.SHIELD2, CF31.SHIELD3, CF32.LC1, CF32.LC2, CF33.SHIELD, CF33.SHIELD1, CF33.SHIELD2, CF33.SHIELD3, CF34.SHIELD, CF34.SHIELD1, CF34.SHIELD2, CF34.SHIELD3, CF35.SHIELD, CF35.SHIELD1, CF35.SHIELD2, CF35.SHIELD3, CF36.LC1, CF36.LC2, CF37.SHIELD, CF37.SHIELD1, CF37.SHIELD2, CF37.SHIELD3, CF38.SHIELD, CF38.SHIELD1, CF38.SHIELD2, CF38.SHIELD3, CF39.SHIELD, CF39.SHIELD1, CF39.SHIELD2, CF39.SHIELD3, CF40.LC1, CF40.LC2, CF41.SHIELD, CF41.SHIELD1, CF41.SHIELD2, CF41.SHIELD3, CF42.SHIELD, CF42.SHIELD1, CF42.SHIELD2, CF42.SHIELD3, CF43.SHIELD, CF43.SHIELD1, CF43.SHIELD2, CF43.SHIELD3, CF44.LC1, CF44.LC2, CF45.SHIELD, CF45.SHIELD1, CF45.SHIELD2, CF45.SHIELD3, CF46.SHIELD, CF46.SHIELD1, CF46.SHIELD2, CF46.SHIELD3, CF47.SHIELD, CF47.SHIELD1, CF47.SHIELD2, CF47.SHIELD3, CF48.LC1, CF48.LC2, CF49.SHIELD, CF49.SHIELD1, CF49.SHIELD2, CF49.SHIELD3, CF50.SHIELD, CF50.SHIELD1, CF50.SHIELD2, CF50.SHIELD3, CF51.SHIELD, CF51.SHIELD1, CF51.SHIELD2, CF51.SHIELD3, CF52.LC1, CF52.LC2, CF53.SHIELD, CF53.SHIELD1, CF53.SHIELD2, CF53.SHIELD3, CF54.SHIELD, CF54.SHIELD1, CF54.SHIELD2, CF54.SHIELD3, CF55.SHIELD, CF55.SHIELD1, CF55.SHIELD2, CF55.SHIELD3, CF56.LC1, CF56.LC2, CF57.SHIELD, CF57.SHIELD1, CF57.SHIELD2, CF57.SHIELD3, CF58.SHIELD, CF58.SHIELD1, CF58.SHIELD2, CF58.SHIELD3, CF59.SHIELD, CF59.SHIELD1, CF59.SHIELD2, CF59.SHIELD3, CF60.LC1, CF60.LC2, CF61.SHIELD, CF61.SHIELD1, CF61.SHIELD2, CF61.SHIELD3, CF62.SHIELD, CF62.SHIELD1, CF62.SHIELD2, CF62.SHIELD3, CF63.SHIELD, CF63.SHIELD1, CF63.SHIELD2, CF63.SHIELD3, CF64.LC1, CF64.LC2, CF65.SHIELD, CF65.SHIELD1, CF65.SHIELD2, CF65.SHIELD3, CF66.SHIELD, CF66.SHIELD1, CF66.SHIELD2, CF66.SHIELD3, CF67.SHIELD, CF67.SHIELD1, CF67.SHIELD2, CF67.SHIELD3, CF68.LC1, CF68.LC2, CF69.SHIELD, CF69.SHIELD1, CF69.SHIELD2, CF69.SHIELD3, CF70.SHIELD, CF70.SHIELD1, CF70.SHIELD2, CF70.SHIELD3, CF71.SHIELD, CF71.SHIELD1, CF71.SHIELD2, CF71.SHIELD3, CF72.LC1, CF72.LC2, CF73.SHIELD, CF73.SHIELD1, CF73.SHIELD2, CF73.SHIELD3, CF74.SHIELD, CF74.SHIELD1, CF74.SHIELD2, CF74.SHIELD3, CF75.SHIELD, CF75.SHIELD1, CF75.SHIELD2, CF75.SHIELD3, CF76.LC1, CF76.LC2, CF77.SHIELD, CF77.SHIELD1, CF77.SHIELD2, CF77.SHIELD3, CF78.SHIELD, CF78.SHIELD1, CF78.SHIELD2, CF78.SHIELD3, CF79.SHIELD, CF79.SHIELD1, CF79.SHIELD2, CF79.SHIELD3, CF80.LC1, CF80.LC2, J10.10, J10.11, J10.12, J10.5, J10.6, J10.9, J10.LC1, J10.LC2, J11.10, J11.11, J11.12, J11.5, J11.6, J11.9, J11.LC1, J11.LC2, J12.10, J12.11, J12.12, J12.5, J12.6, J12.9, J12.LC1, J12.LC2, J13.10, J13.11, J13.12, J13.5, J13.6, J13.9, J13.LC1, J13.LC2, J15.10, J15.11, J15.12, J15.5, J15.6, J15.9, J15.LC1, J15.LC2, J16.10, J16.11, J16.12, J16.5, J16.6, J16.9, J16.LC1, J16.LC2, J17.10, J17.11, J17.12, J17.5, J17.6, J17.9, J17.LC1, J17.LC2, J18.10, J18.11, J18.12, J18.5, J18.6, J18.9, J18.LC1, J18.LC2, J19.10, J19.11, J19.12, J19.5, J19.6, J19.9, J19.LC1, J19.LC2, J8.10, J8.11, J8.12, J8.5, J8.6, J8.9, J8.LC1, J8.LC2, J9.10, J9.11, J9.12, J9.5, J9.6, J9.9, J9.LC1, J9.LC2
- net VBUS: now also J10.13, J10.14, J10.15, J10.16, J11.13, J11.14, J11.15, J11.16, J12.13, J12.14, J12.15, J12.16, J13.13, J13.14, J13.15, J13.16, J15.13, J15.14, J15.15, J15.16, J16.13, J16.14, J16.15, J16.16, J17.13, J17.14, J17.15, J17.16, J18.13, J18.14, J18.15, J18.16, J19.13, J19.14, J19.15, J19.16, J8.13, J8.14, J8.15, J8.16, J9.13, J9.14, J9.15, J9.16

Commit message: Backplane v1.0. Finally. Uses SMPM RF connectors.
Parts:
- removed CF1, CF10, CF11, CF13, CF14, CF15, CF17, CF18, CF19, CF2, CF21, CF22, CF23, CF25, CF26, CF27, CF29, CF3, CF30, CF31, CF33, CF34, CF35, CF37, CF38, CF39, CF4, CF41, CF42, CF43, CF45, CF46, CF47, CF49, CF5, CF50, CF51, CF53, CF54, CF55, CF57, CF58, CF59, CF6, CF61, CF62, CF63, CF65, CF66, CF67, CF69, CF70, CF71, CF73, CF74, CF75, CF77, CF78, CF79, CF9: ORESAT-BACKPLANE-TO-UT-047, J-Cinch-MMCX-135-3701-211-to-UT-047:ORESAT-BACKPLANE-TO-UT-047
- added CM1.1, CM1.2, CM1.3, CM10.1, CM10.2, CM10.3, CM11.1, CM11.2, CM11.3, CM12.1, CM12.2, CM12.3, CM13.1, CM13.2, CM13.3, CM14.1, CM14.2, CM14.3, CM15.1, CM15.2, CM15.3, CM16.1, CM16.2, CM16.3, CM17.1, CM17.2, CM17.3, CM18.1, CM18.2, CM18.3, CM19.1, CM19.2, CM19.3, CM2.1, CM2.2, CM2.3, CM20.1, CM20.2, CM20.3, CM3.1, CM3.2, CM3.3, CM4.1, CM4.2, CM4.3, CM5.1, CM5.2, CM5.3, CM6.1, CM6.2, CM6.3, CM7.1, CM7.2, CM7.3, CM8.1, CM8.2, CM8.3, CM9.1, CM9.2, CM9.3: J-MOLEX-SMPM-73300-0111X, J-Molex-SMPM-73300-011x:J-MOLEX-SMPM-73300-0111X
- renumbered CF12 to CF18.1, CF16 to CF17.1, CF20 to CF16.1, CF24 to CF15.1, CF28 to CF14.1, CF32 to CF13.1, CF36 to CF12.1, CF40 to CF11.1, CF44 to CF10.1, CF48 to CF9.1, CF52 to CF8.1, CF56 to CF7.1, CF60 to CF6.1, CF64 to CF5.1, CF68 to CF4.1, CF7 to CF19.1, CF72 to CF3.1, CF76 to CF2.1, CF8 to CF20.1, CF80 to CF1.1, J10 to CF11.2, J11 to CF10.2, J12 to CF9.2, J13 to CF8.2, J14 to CF7.2, J15 to CF6.2, J16 to CF5.2, J17 to CF4.2, J18 to CF3.2, J19 to CF2.2, J2 to CF19.2, J3 to CF18.2, J4 to CF17.2, J5 to CF16.2, J6 to CF15.2, J7 to CF14.2, J8 to CF13.2, J9 to CF12.2
Connections:
- net GND: now also CM1.1.SHIELD, CM1.1.SHIELD1, CM1.1.SHIELD2, CM1.1.SHIELD3, CM1.1.SHIELD4, CM1.1.SHIELD5, CM1.2.SHIELD, CM1.2.SHIELD1, CM1.2.SHIELD2, CM1.2.SHIELD3, CM1.2.SHIELD4, CM1.2.SHIELD5, CM1.3.SHIELD, CM1.3.SHIELD1, CM1.3.SHIELD2, CM1.3.SHIELD3, CM1.3.SHIELD4, CM1.3.SHIELD5, CM10.1.SHIELD, CM10.1.SHIELD1, CM10.1.SHIELD2, CM10.1.SHIELD3, CM10.1.SHIELD4, CM10.1.SHIELD5, CM10.2.SHIELD, CM10.2.SHIELD1, CM10.2.SHIELD2, CM10.2.SHIELD3, CM10.2.SHIELD4, CM10.2.SHIELD5, CM10.3.SHIELD, CM10.3.SHIELD1, CM10.3.SHIELD2, CM10.3.SHIELD3, CM10.3.SHIELD4, CM10.3.SHIELD5, CM11.1.SHIELD, CM11.1.SHIELD1, CM11.1.SHIELD2, CM11.1.SHIELD3, CM11.1.SHIELD4, CM11.1.SHIELD5, CM11.2.SHIELD, CM11.2.SHIELD1, CM11.2.SHIELD2, CM11.2.SHIELD3, CM11.2.SHIELD4, CM11.2.SHIELD5, CM11.3.SHIELD, CM11.3.SHIELD1, CM11.3.SHIELD2, CM11.3.SHIELD3, CM11.3.SHIELD4, CM11.3.SHIELD5, CM12.1.SHIELD, CM12.1.SHIELD1, CM12.1.SHIELD2, CM12.1.SHIELD3, CM12.1.SHIELD4, CM12.1.SHIELD5, CM12.2.SHIELD, CM12.2.SHIELD1, CM12.2.SHIELD2, CM12.2.SHIELD3, CM12.2.SHIELD4, CM12.2.SHIELD5, CM12.3.SHIELD, CM12.3.SHIELD1, CM12.3.SHIELD2, CM12.3.SHIELD3, CM12.3.SHIELD4, CM12.3.SHIELD5, CM13.1.SHIELD, CM13.1.SHIELD1, CM13.1.SHIELD2, CM13.1.SHIELD3, CM13.1.SHIELD4, CM13.1.SHIELD5, CM13.2.SHIELD, CM13.2.SHIELD1, CM13.2.SHIELD2, CM13.2.SHIELD3, CM13.2.SHIELD4, CM13.2.SHIELD5, CM13.3.SHIELD, CM13.3.SHIELD1, CM13.3.SHIELD2, CM13.3.SHIELD3, CM13.3.SHIELD4, CM13.3.SHIELD5, CM14.1.SHIELD, CM14.1.SHIELD1, CM14.1.SHIELD2, CM14.1.SHIELD3, CM14.1.SHIELD4, CM14.1.SHIELD5, CM14.2.SHIELD, CM14.2.SHIELD1, CM14.2.SHIELD2, CM14.2.SHIELD3, CM14.2.SHIELD4, CM14.2.SHIELD5, CM14.3.SHIELD, CM14.3.SHIELD1, CM14.3.SHIELD2, CM14.3.SHIELD3, CM14.3.SHIELD4, CM14.3.SHIELD5, CM15.1.SHIELD, CM15.1.SHIELD1, CM15.1.SHIELD2, CM15.1.SHIELD3, CM15.1.SHIELD4, CM15.1.SHIELD5, CM15.2.SHIELD, CM15.2.SHIELD1, CM15.2.SHIELD2, CM15.2.SHIELD3, CM15.2.SHIELD4, CM15.2.SHIELD5, CM15.3.SHIELD, CM15.3.SHIELD1, CM15.3.SHIELD2, CM15.3.SHIELD3, CM15.3.SHIELD4, CM15.3.SHIELD5, CM16.1.SHIELD, CM16.1.SHIELD1, CM16.1.SHIELD2, CM16.1.SHIELD3, CM16.1.SHIELD4, CM16.1.SHIELD5, CM16.2.SHIELD, CM16.2.SHIELD1, CM16.2.SHIELD2, CM16.2.SHIELD3, CM16.2.SHIELD4, CM16.2.SHIELD5, CM16.3.SHIELD, CM16.3.SHIELD1, CM16.3.SHIELD2, CM16.3.SHIELD3, CM16.3.SHIELD4, CM16.3.SHIELD5, CM17.1.SHIELD, CM17.1.SHIELD1, CM17.1.SHIELD2, CM17.1.SHIELD3, CM17.1.SHIELD4, CM17.1.SHIELD5, CM17.2.SHIELD, CM17.2.SHIELD1, CM17.2.SHIELD2, CM17.2.SHIELD3, CM17.2.SHIELD4, CM17.2.SHIELD5, CM17.3.SHIELD, CM17.3.SHIELD1, CM17.3.SHIELD2, CM17.3.SHIELD3, CM17.3.SHIELD4, CM17.3.SHIELD5, CM18.1.SHIELD, CM18.1.SHIELD1, CM18.1.SHIELD2, CM18.1.SHIELD3, CM18.1.SHIELD4, CM18.1.SHIELD5, CM18.2.SHIELD, CM18.2.SHIELD1, CM18.2.SHIELD2, CM18.2.SHIELD3, CM18.2.SHIELD4, CM18.2.SHIELD5, CM18.3.SHIELD, CM18.3.SHIELD1, CM18.3.SHIELD2, CM18.3.SHIELD3, CM18.3.SHIELD4, CM18.3.SHIELD5, CM19.1.SHIELD, CM19.1.SHIELD1, CM19.1.SHIELD2, CM19.1.SHIELD3, CM19.1.SHIELD4, CM19.1.SHIELD5, CM19.2.SHIELD, CM19.2.SHIELD1, CM19.2.SHIELD2, CM19.2.SHIELD3, CM19.2.SHIELD4, CM19.2.SHIELD5, CM19.3.SHIELD, CM19.3.SHIELD1, CM19.3.SHIELD2, CM19.3.SHIELD3, CM19.3.SHIELD4, CM19.3.SHIELD5, CM2.1.SHIELD, CM2.1.SHIELD1, CM2.1.SHIELD2, CM2.1.SHIELD3, CM2.1.SHIELD4, CM2.1.SHIELD5, CM2.2.SHIELD, CM2.2.SHIELD1, CM2.2.SHIELD2, CM2.2.SHIELD3, CM2.2.SHIELD4, CM2.2.SHIELD5, CM2.3.SHIELD, CM2.3.SHIELD1, CM2.3.SHIELD2, CM2.3.SHIELD3, CM2.3.SHIELD4, CM2.3.SHIELD5, CM20.1.SHIELD, CM20.1.SHIELD1, CM20.1.SHIELD2, CM20.1.SHIELD3, CM20.1.SHIELD4, CM20.1.SHIELD5, CM20.2.SHIELD, CM20.2.SHIELD1, CM20.2.SHIELD2, CM20.2.SHIELD3, CM20.2.SHIELD4, CM20.2.SHIELD5, CM20.3.SHIELD, CM20.3.SHIELD1, CM20.3.SHIELD2, CM20.3.SHIELD3, CM20.3.SHIELD4, CM20.3.SHIELD5, CM3.1.SHIELD, CM3.1.SHIELD1, CM3.1.SHIELD2, CM3.1.SHIELD3, CM3.1.SHIELD4, CM3.1.SHIELD5, CM3.2.SHIELD, CM3.2.SHIELD1, CM3.2.SHIELD2, CM3.2.SHIELD3, CM3.2.SHIELD4, CM3.2.SHIELD5, CM3.3.SHIELD, CM3.3.SHIELD1, CM3.3.SHIELD2, CM3.3.SHIELD3, CM3.3.SHIELD4, CM3.3.SHIELD5, CM4.1.SHIELD, CM4.1.SHIELD1, CM4.1.SHIELD2, CM4.1.SHIELD3, CM4.1.SHIELD4, CM4.1.SHIELD5, CM4.2.SHIELD, CM4.2.SHIELD1, CM4.2.SHIELD2, CM4.2.SHIELD3, CM4.2.SHIELD4, CM4.2.SHIELD5, CM4.3.SHIELD, CM4.3.SHIELD1, CM4.3.SHIELD2, CM4.3.SHIELD3, CM4.3.SHIELD4, CM4.3.SHIELD5, CM5.1.SHIELD, CM5.1.SHIELD1, CM5.1.SHIELD2, CM5.1.SHIELD3, CM5.1.SHIELD4, CM5.1.SHIELD5, CM5.2.SHIELD, CM5.2.SHIELD1, CM5.2.SHIELD2, CM5.2.SHIELD3, CM5.2.SHIELD4, CM5.2.SHIELD5, CM5.3.SHIELD, CM5.3.SHIELD1, CM5.3.SHIELD2, CM5.3.SHIELD3, CM5.3.SHIELD4, CM5.3.SHIELD5, CM6.1.SHIELD, CM6.1.SHIELD1, CM6.1.SHIELD2, CM6.1.SHIELD3, CM6.1.SHIELD4, CM6.1.SHIELD5, CM6.2.SHIELD, CM6.2.SHIELD1, CM6.2.SHIELD2, CM6.2.SHIELD3, CM6.2.SHIELD4, CM6.2.SHIELD5, CM6.3.SHIELD, CM6.3.SHIELD1, CM6.3.SHIELD2, CM6.3.SHIELD3, CM6.3.SHIELD4, CM6.3.SHIELD5, CM7.1.SHIELD, CM7.1.SHIELD1, CM7.1.SHIELD2, CM7.1.SHIELD3, CM7.1.SHIELD4, CM7.1.SHIELD5, CM7.2.SHIELD, CM7.2.SHIELD1, CM7.2.SHIELD2, CM7.2.SHIELD3, CM7.2.SHIELD4, CM7.2.SHIELD5, CM7.3.SHIELD, CM7.3.SHIELD1, CM7.3.SHIELD2, CM7.3.SHIELD3, CM7.3.SHIELD4, CM7.3.SHIELD5, CM8.1.SHIELD, CM8.1.SHIELD1, CM8.1.SHIELD2, CM8.1.SHIELD3, CM8.1.SHIELD4, CM8.1.SHIELD5, CM8.2.SHIELD, CM8.2.SHIELD1, CM8.2.SHIELD2, CM8.2.SHIELD3, CM8.2.SHIELD4, CM8.2.SHIELD5, CM8.3.SHIELD, CM8.3.SHIELD1, CM8.3.SHIELD2, CM8.3.SHIELD3, CM8.3.SHIELD4, CM8.3.SHIELD5, CM9.1.SHIELD, CM9.1.SHIELD1, CM9.1.SHIELD2, CM9.1.SHIELD3, CM9.1.SHIELD4, CM9.1.SHIELD5, CM9.2.SHIELD, CM9.2.SHIELD1, CM9.2.SHIELD2, CM9.2.SHIELD3, CM9.2.SHIELD4, CM9.2.SHIELD5, CM9.3.SHIELD, CM9.3.SHIELD1, CM9.3.SHIELD2, CM9.3.SHIELD3, CM9.3.SHIELD4, CM9.3.SHIELD5; no longer CF1.SHIELD, CF1.SHIELD1, CF1.SHIELD2, CF1.SHIELD3, CF10.SHIELD, CF10.SHIELD1, CF10.SHIELD2, CF10.SHIELD3, CF11.SHIELD, CF11.SHIELD1, CF11.SHIELD2, CF11.SHIELD3, CF13.SHIELD, CF13.SHIELD1, CF13.SHIELD2, CF13.SHIELD3, CF14.SHIELD, CF14.SHIELD1, CF14.SHIELD2, CF14.SHIELD3, CF15.SHIELD, CF15.SHIELD1, CF15.SHIELD2, CF15.SHIELD3, CF17.SHIELD, CF17.SHIELD1, CF17.SHIELD2, CF17.SHIELD3, CF18.SHIELD, CF18.SHIELD1, CF18.SHIELD2, CF18.SHIELD3, CF19.SHIELD, CF19.SHIELD1, CF19.SHIELD2, CF19.SHIELD3, CF2.SHIELD, CF2.SHIELD1, CF2.SHIELD2, CF2.SHIELD3, CF21.SHIELD, CF21.SHIELD1, CF21.SHIELD2, CF21.SHIELD3, CF22.SHIELD, CF22.SHIELD1, CF22.SHIELD2, CF22.SHIELD3, CF23.SHIELD, CF23.SHIELD1, CF23.SHIELD2, CF23.SHIELD3, CF25.SHIELD, CF25.SHIELD1, CF25.SHIELD2, CF25.SHIELD3, CF26.SHIELD, CF26.SHIELD1, CF26.SHIELD2, CF26.SHIELD3, CF27.SHIELD, CF27.SHIELD1, CF27.SHIELD2, CF27.SHIELD3, CF29.SHIELD, CF29.SHIELD1, CF29.SHIELD2, CF29.SHIELD3, CF3.SHIELD, CF3.SHIELD1, CF3.SHIELD2, CF3.SHIELD3, CF30.SHIELD, CF30.SHIELD1, CF30.SHIELD2, CF30.SHIELD3, CF31.SHIELD, CF31.SHIELD1, CF31.SHIELD2, CF31.SHIELD3, CF33.SHIELD, CF33.SHIELD1, CF33.SHIELD2, CF33.SHIELD3, CF34.SHIELD, CF34.SHIELD1, CF34.SHIELD2, CF34.SHIELD3, CF35.SHIELD, CF35.SHIELD1, CF35.SHIELD2, CF35.SHIELD3, CF37.SHIELD, CF37.SHIELD1, CF37.SHIELD2, CF37.SHIELD3, CF38.SHIELD, CF38.SHIELD1, CF38.SHIELD2, CF38.SHIELD3, CF39.SHIELD, CF39.SHIELD1, CF39.SHIELD2, CF39.SHIELD3, CF4.SHIELD, CF4.SHIELD1, CF4.SHIELD2, CF4.SHIELD3, CF41.SHIELD, CF41.SHIELD1, CF41.SHIELD2, CF41.SHIELD3, CF42.SHIELD, CF42.SHIELD1, CF42.SHIELD2, CF42.SHIELD3, CF43.SHIELD, CF43.SHIELD1, CF43.SHIELD2, CF43.SHIELD3, CF45.SHIELD, CF45.SHIELD1, CF45.SHIELD2, CF45.SHIELD3, CF46.SHIELD, CF46.SHIELD1, CF46.SHIELD2, CF46.SHIELD3, CF47.SHIELD, CF47.SHIELD1, CF47.SHIELD2, CF47.SHIELD3, CF49.SHIELD, CF49.SHIELD1, CF49.SHIELD2, CF49.SHIELD3, CF5.SHIELD, CF5.SHIELD1, CF5.SHIELD2, CF5.SHIELD3, CF50.SHIELD, CF50.SHIELD1, CF50.SHIELD2, CF50.SHIELD3, CF51.SHIELD, CF51.SHIELD1, CF51.SHIELD2, CF51.SHIELD3, CF53.SHIELD, CF53.SHIELD1, CF53.SHIELD2, CF53.SHIELD3, CF54.SHIELD, CF54.SHIELD1, CF54.SHIELD2, CF54.SHIELD3, CF55.SHIELD, CF55.SHIELD1, CF55.SHIELD2, CF55.SHIELD3, CF57.SHIELD, CF57.SHIELD1, CF57.SHIELD2, CF57.SHIELD3, CF58.SHIELD, CF58.SHIELD1, CF58.SHIELD2, CF58.SHIELD3, CF59.SHIELD, CF59.SHIELD1, CF59.SHIELD2, CF59.SHIELD3, CF6.SHIELD, CF6.SHIELD1, CF6.SHIELD2, CF6.SHIELD3, CF61.SHIELD, CF61.SHIELD1, CF61.SHIELD2, CF61.SHIELD3, CF62.SHIELD, CF62.SHIELD1, CF62.SHIELD2, CF62.SHIELD3, CF63.SHIELD, CF63.SHIELD1, CF63.SHIELD2, CF63.SHIELD3, CF65.SHIELD, CF65.SHIELD1, CF65.SHIELD2, CF65.SHIELD3, CF66.SHIELD, CF66.SHIELD1, CF66.SHIELD2, CF66.SHIELD3, CF67.SHIELD, CF67.SHIELD1, CF67.SHIELD2, CF67.SHIELD3, CF69.SHIELD, CF69.SHIELD1, CF69.SHIELD2, CF69.SHIELD3, CF70.SHIELD, CF70.SHIELD1, CF70.SHIELD2, CF70.SHIELD3, CF71.SHIELD, CF71.SHIELD1, CF71.SHIELD2, CF71.SHIELD3, CF73.SHIELD, CF73.SHIELD1, CF73.SHIELD2, CF73.SHIELD3, CF74.SHIELD, CF74.SHIELD1, CF74.SHIELD2, CF74.SHIELD3, CF75.SHIELD, CF75.SHIELD1, CF75.SHIELD2, CF75.SHIELD3, CF77.SHIELD, CF77.SHIELD1, CF77.SHIELD2, CF77.SHIELD3, CF78.SHIELD, CF78.SHIELD1, CF78.SHIELD2, CF78.SHIELD3, CF79.SHIELD, CF79.SHIELD1, CF79.SHIELD2, CF79.SHIELD3, CF9.SHIELD, CF9.SHIELD1, CF9.SHIELD2, CF9.SHIELD3
