File: 1u/KiCad/oresat0-1u-backplane/Slot_4.kicad_sch (KiCad schematic)
At the start: 3 parts

Commit message: Fixed DRC errors and warnings
Parts:
- C8: value (none) -> 10u 25V; footprint (none) -> oresat0-1u-backplane:1206-B
- CF4.2: value (none) -> SFM-120-X1-XXX-D; footprint (none) -> oresat0-1u-backplane:SFM-120-X1-XXX-D
- CM4.1: value (none) -> J-MOLEX-SMPM-73300-0111X; footprint (none) -> oresat-footprints:J-MOLEX-SMPM-73300-0111X-long; symbol oresat0-1u-backplane-eagle-import:J-MOLEX-SMPM-73300-0111X -> J-MOLEX-SMPM-73300-0111X:J-MOLEX-SMPM-73300-0111X_1
Connections:
- net GND: now also CM4.1.GND (SHIELD1); no longer CM4.1.P$1 (SHIELD1), CM4.1.P$2 (SHIELD1), CM4.1.P$3 (SHIELD1), CM4.1.P$4 (SHIELD1)
Changed lines of the file:
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@@
       (effects (font (size 1.27 1.0795)) (justify left bottom))
     )
-    (property "Value" "" (id 1) (at 82.55 71.12 0)
+    (property "Value" "SFM-120-X1-XXX-D" (id 1) (at 82.55 71.12 0)
       (effects (font (size 1.27 1.0795)) (justify left bottom))
     )
-    (property "Footprint" "" (id 2) (at 85.09 120.65 0)
+    (property "Footprint" "oresat0-1u-backplane:SFM-120-X1-XXX-D" (id 2) (at 85.09 120.65 0)
       (effects (font (size 1.27 1.27)) hide)
     )
@@
     (pin "LC2")
   )
-  (symbol (lib_id "oresat0-1u-backplane-eagle-import:J-MOLEX-SMPM-73300-0111X") (at 196.85 95.25 0) (unit 1)
+  (symbol (lib_id "J-MOLEX-SMPM-73300-0111X:J-MOLEX-SMPM-73300-0111X_1") (at 196.85 95.25 0) (unit 1)
     (in_bom yes) (on_board yes)
     (property "Reference" "CM4.1" (id 0) (at 200.66 99.06 0)
       (effects (font (size 1.778 1.5113) bold) (justify left bottom))
     )
-    (property "Value" "" (id 1) (at 200.66 101.6 0)
+    (property "Value" "J-MOLEX-SMPM-73300-0111X" (id 1) (at 200.66 101.6 0)
       (effects (font (size 1.778 1.5113) bold) (justify left bottom))
     )
-    (property "Footprint" "" (id 2) (at 196.85 95.25 0)
+    (property "Footprint" "oresat-footprints:J-MOLEX-SMPM-73300-0111X-long" (id 2) (at 196.85 95.25 0)
       (effects (font (size 1.27 1.27)) hide)
     )
@@
       (effects (font (size 1.27 1.27)) hide)
     )
-    (pin "P$1")
-    (pin "P$2")
-    (pin "P$3")
-    (pin "P$4")
+    (pin "GND")
     (pin "RF-DOWN")
   )
@@
       (effects (font (size 1.778 1.5113)) (justify left bottom))
     )
-    (property "Value" "" (id 1) (at 118.364 144.399 0)
+    (property "Value" "10u 25V" (id 1) (at 118.364 144.399 0)
       (effects (font (size 1.778 1.5113)) (justify left bottom))
     )
-    (property "Footprint" "" (id 2) (at 116.84 139.7 0)
+    (property "Footprint" "oresat0-1u-backplane:1206-B" (id 2) (at 116.84 139.7 0)
       (effects (font (size 1.27 1.27)) hide)
     )
@@
   (symbol (lib_id "oresat0-1u-backplane-eagle-import:GND") (at 97.79 184.15 0) (unit 1)
     (in_bom yes) (on_board yes)
-    (property "Reference" "#GND97" (id 0) (at 97.79 184.15 0)
+    (property "Reference" "#GND097" (id 0) (at 97.79 184.15 0)
       (effects (font (size 1.27 1.27)) hide)
     )
-    (property "Value" "" (id 1) (at 97.79 184.15 0)
+    (property "Value" "GND" (id 1) (at 97.79 184.15 0)
       (effects (font (size 1.27 1.27)) hide)
     )
-    (property "Footprint" "" (id 2) (at 97.79 184.15 0)
+    (property "Footprint" "oresat0-1u-backplane:" (id 2) (at 97.79 184.15 0)
       (effects (font (size 1.27 1.27)) hide)
     )
@@
     (pin "1")
   )
-  (symbol (lib_id "oresat0-1u-backplane-eagle-import:FRAME_A_L") (at 17.78 233.68 0) (unit 1)
+  (symbol (lib_id "oresat0-1u-backplane-eagle-import:GND") (at 196.85 100.33 0) (unit 1)
     (in_bom yes) (on_board yes)
-    (property "Reference" "#FRAME17" (id 0) (at 17.78 233.68 0)
+    (property "Reference" "#GND05" (id 0) (at 196.85 100.33 0)
       (effects (font (size 1.27 1.27)) hide)
     )
-    (property "Value" "" (id 1) (at 17.78 233.68 0)
+    (property "Value" "GND" (id 1) (at 196.85 100.33 0)
       (effects (font (size 1.27 1.27)) hide)
     )
-    (property "Footprint" "" (id 2) (at 17.78 233.68 0)
+    (property "Footprint" "oresat0-1u-backplane:" (id 2) (at 196.85 100.33 0)
       (effects (font (size 1.27 1.27)) hide)
     )
-    (property "Datasheet" "" (id 3) (at 17.78 233.68 0)
-      (effects (font (size 1.27 1.27)) hide)
-    )
-  )
-  (symbol (lib_id "oresat0-1u-backplane-eagle-import:FRAME_A_L") (at 190.5 233.68 0) (unit 2)
-    (in_bom yes) (on_board yes)
-    (property "Reference" "#FRAME17" (id 0) (at 190.5 233.68 0)
-      (effects (font (size 1.27 1.27)) hide)
-    )
-    (property "Value" "" (id 1) (at 190.5 233.68 0)
-      (effects (font (size 1.27 1.27)) hide)
-    )
-    (property "Footprint" "" (id 2) (at 190.5 233.68 0)
-      (effects (font (size 1.27 1.27)) hide)
-    )
-    (property "Datasheet" "" (id 3) (at 190.5 233.68 0)
-      (effects (font (size 1.27 1.27)) hide)
-    )
-  )
-  (symbol (lib_id "oresat0-1u-backplane-eagle-import:GND") (at 196.85 100.33 0) (unit 1)
-    (in_bom yes) (on_board yes)
-    (property "Reference" "#GND5" (id 0) (at 196.85 100.33 0)
-      (effects (font (size 1.27 1.27)) hide)
-    )
-    (property "Value" "" (id 1) (at 196.85 100.33 0)
-      (effects (font (size 1.27 1.27)) hide)
-    )
-    (property "Footprint" "" (id 2) (at 196.85 100.33 0)
-      (effects (font (size 1.27 1.27)) hide)
-    )
