File: 1u/KiCad/oresat0-1u-backplane/Slot_5.kicad_sch (KiCad schematic)
At the start: 3 parts

Commit message: Fixed DRC errors and warnings
Parts:
- C9: value (none) -> 10u 25V; footprint (none) -> oresat0-1u-backplane:1206-B
- CF5.2: value (none) -> SFM-120-X1-XXX-D; footprint (none) -> oresat0-1u-backplane:SFM-120-X1-XXX-D
- J2: value (none) -> M55-6001642R; footprint (none) -> oresat0-1u-backplane:CONN_M55-6001642R_HRW
Changed lines of the file:
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@@
   (symbol (lib_id "oresat0-1u-backplane-eagle-import:GND") (at 69.85 175.26 0) (unit 1)
     (in_bom yes) (on_board yes)
-    (property "Reference" "#GND91" (id 0) (at 69.85 175.26 0)
+    (property "Reference" "#GND091" (id 0) (at 69.85 175.26 0)
       (effects (font (size 1.27 1.27)) hide)
     )
-    (property "Value" "" (id 1) (at 69.85 175.26 0)
+    (property "Value" "GND" (id 1) (at 69.85 175.26 0)
       (effects (font (size 1.27 1.27)) hide)
     )
-    (property "Footprint" "" (id 2) (at 69.85 175.26 0)
+    (property "Footprint" "oresat0-1u-backplane:" (id 2) (at 69.85 175.26 0)
       (effects (font (size 1.27 1.27)) hide)
     )
@@
       (effects (font (size 1.778 1.5113)) (justify left bottom))
     )
-    (property "Value" "" (id 1) (at 210.82 92.71 0)
+    (property "Value" "M55-6001642R" (id 1) (at 210.82 92.71 0)
       (effects (font (size 1.778 1.5113)) (justify left bottom))
     )
-    (property "Footprint" "" (id 2) (at 215.9 114.3 0)
+    (property "Footprint" "oresat0-1u-backplane:CONN_M55-6001642R_HRW" (id 2) (at 215.9 114.3 0)
       (effects (font (size 1.27 1.27)) hide)
     )
@@
       (effects (font (size 1.778 1.5113)) (justify left bottom))
     )
-    (property "Value" "" (id 1) (at 91.694 134.239 0)
+    (property "Value" "10u 25V" (id 1) (at 91.694 134.239 0)
       (effects (font (size 1.778 1.5113)) (justify left bottom))
     )
-    (property "Footprint" "" (id 2) (at 90.17 129.54 0)
+    (property "Footprint" "oresat0-1u-backplane:1206-B" (id 2) (at 90.17 129.54 0)
       (effects (font (size 1.27 1.27)) hide)
     )
@@
     (pin "2")
   )
-  (symbol (lib_id "oresat0-1u-backplane-eagle-import:FRAME_A_L") (at 190.5 233.68 0) (unit 2)
+  (symbol (lib_id "oresat0-1u-backplane-eagle-import:GND") (at 214.63 140.97 0) (unit 1)
     (in_bom yes) (on_board yes)
-    (property "Reference" "#FRAME16" (id 0) (at 190.5 233.68 0)
+    (property "Reference" "#GND07" (id 0) (at 214.63 140.97 0)
       (effects (font (size 1.27 1.27)) hide)
     )
-    (property "Value" "" (id 1) (at 190.5 233.68 0)
+    (property "Value" "GND" (id 1) (at 214.63 140.97 0)
       (effects (font (size 1.27 1.27)) hide)
     )
-    (property "Footprint" "" (id 2) (at 190.5 233.68 0)
-      (effects (font (size 1.27 1.27)) hide)
-    )
-    (property "Datasheet" "" (id 3) (at 190.5 233.68 0)
-      (effects (font (size 1.27 1.27)) hide)
-    )
-  )
-  (symbol (lib_id "oresat0-1u-backplane-eagle-import:GND") (at 214.63 140.97 0) (unit 1)
-    (in_bom yes) (on_board yes)
-    (property "Reference" "#GND7" (id 0) (at 214.63 140.97 0)
-      (effects (font (size 1.27 1.27)) hide)
-    )
-    (property "Value" "" (id 1) (at 214.63 140.97 0)
-      (effects (font (size 1.27 1.27)) hide)
-    )
-    (property "Footprint" "" (id 2) (at 214.63 140.97 0)
+    (property "Footprint" "oresat0-1u-backplane:" (id 2) (at 214.63 140.97 0)
       (effects (font (size 1.27 1.27)) hide)
     )
@@
       (effects (font (size 1.27 1.0795)) (justify left bottom))
     )
-    (property "Value" "" (id 1) (at 54.61 62.23 0)
+    (property "Value" "SFM-120-X1-XXX-D" (id 1) (at 54.61 62.23 0)
       (effects (font (size 1.27 1.0795)) (justify left bottom))
     )
-    (property "Footprint" "" (id 2) (at 57.15 111.76 0)
+    (property "Footprint" "oresat0-1u-backplane:SFM-120-X1-XXX-D" (id 2) (at 57.15 111.76 0)
       (effects (font (size 1.27 1.27)) hide)
     )
@@
     (pin "LC2")
   )
-  (symbol (lib_id "oresat0-1u-backplane-eagle-import:FRAME_A_L") (at 17.78 233.68 0) (unit 1)
-    (in_bom yes) (on_board yes)
-    (property "Reference" "#FRAME16" (id 0) (at 17.78 233.68 0)
-      (effects (font (size 1.27 1.27)) hide)
-    )
-    (property "Value" "" (id 1) (at 17.78 233.68 0)
-      (effects (font (size 1.27 1.27)) hide)
-    )
-    (property "Footprint" "" (id 2) (at 17.78 233.68 0)
-      (effects (font (size 1.27 1.27)) hide)
-    )
-    (property "Datasheet" "" (id 3) (at 17.78 233.68 0)
-      (effects (font (size 1.27 1.27)) hide)
-    )
-  )
 )
