File: 1u/KiCad/oresat0-1u-backplane/Slot_8.kicad_sch (KiCad schematic)
At the start: 8 parts

Commit message: Fixed DRC errors and warnings
Parts:
- C3, C4: value (none) -> 1n; footprint (none) -> oresat0-1u-backplane:.0603-C-NOSILK
- R10, R9: value (none) -> 0; footprint (none) -> oresat0-1u-backplane:.0603-B-NOSILK
- R5, R6, R7, R8: value (none) -> NP/60.4; footprint (none) -> oresat0-1u-backplane:1206-C
Changed lines of the file:
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@@
       (effects (font (size 1.778 1.5113)) (justify left bottom))
     )
-    (property "Value" "" (id 1) (at 119.38 115.57 0)
+    (property "Value" "0" (id 1) (at 119.38 115.57 0)
       (effects (font (size 1.778 1.5113)) (justify left bottom))
     )
-    (property "Footprint" "" (id 2) (at 120.65 118.11 0)
+    (property "Footprint" "oresat0-1u-backplane:.0603-B-NOSILK" (id 2) (at 120.65 118.11 0)
       (effects (font (size 1.27 1.27)) hide)
     )
@@
       (effects (font (size 1.778 1.5113)) (justify left bottom))
     )
-    (property "Value" "" (id 1) (at 157.734 102.489 0)
+    (property "Value" "1n" (id 1) (at 157.734 102.489 0)
       (effects (font (size 1.778 1.5113)) (justify left bottom))
     )
-    (property "Footprint" "" (id 2) (at 156.21 97.79 0)
+    (property "Footprint" "oresat0-1u-backplane:.0603-C-NOSILK" (id 2) (at 156.21 97.79 0)
       (effects (font (size 1.27 1.27)) hide)
     )
@@
       (effects (font (size 1.778 1.5113)) (justify left bottom))
     )
-    (property "Value" "" (id 1) (at 127 115.57 0)
+    (property "Value" "0" (id 1) (at 127 115.57 0)
       (effects (font (size 1.778 1.5113)) (justify left bottom))
     )
-    (property "Footprint" "" (id 2) (at 128.27 118.11 0)
+    (property "Footprint" "oresat0-1u-backplane:.0603-B-NOSILK" (id 2) (at 128.27 118.11 0)
       (effects (font (size 1.27 1.27)) hide)
     )
@@
   (symbol (lib_id "oresat0-1u-backplane-eagle-import:GND") (at 156.21 105.41 0) (unit 1)
     (in_bom yes) (on_board yes)
-    (property "Reference" "#GND18" (id 0) (at 156.21 105.41 0)
+    (property "Reference" "#GND018" (id 0) (at 156.21 105.41 0)
       (effects (font (size 1.27 1.27)) hide)
     )
-    (property "Value" "" (id 1) (at 156.21 105.41 0)
+    (property "Value" "GND" (id 1) (at 156.21 105.41 0)
       (effects (font (size 1.27 1.27)) hide)
     )
-    (property "Footprint" "" (id 2) (at 156.21 105.41 0)
+    (property "Footprint" "oresat0-1u-backplane:" (id 2) (at 156.21 105.41 0)
       (effects (font (size 1.27 1.27)) hide)
     )
@@
     (pin "1")
   )
-  (symbol (lib_id "oresat0-1u-backplane-eagle-import:FRAME_A_L") (at 190.5 233.68 0) (unit 2)
-    (in_bom yes) (on_board yes)
-    (property "Reference" "#FRAME13" (id 0) (at 190.5 233.68 0)
-      (effects (font (size 1.27 1.27)) hide)
-    )
-    (property "Value" "" (id 1) (at 190.5 233.68 0)
-      (effects (font (size 1.27 1.27)) hide)
-    )
-    (property "Footprint" "" (id 2) (at 190.5 233.68 0)
-      (effects (font (size 1.27 1.27)) hide)
-    )
-    (property "Datasheet" "" (id 3) (at 190.5 233.68 0)
-      (effects (font (size 1.27 1.27)) hide)
-    )
-  )
   (symbol (lib_id "oresat0-1u-backplane-eagle-import:R-US_1206-C") (at 146.05 130.81 0) (unit 1)
     (in_bom yes) (on_board yes)
@@
       (effects (font (size 1.778 1.5113)) (justify left bottom))
     )
-    (property "Value" "" (id 1) (at 147.32 129.032 0)
+    (property "Value" "NP/60.4" (id 1) (at 147.32 129.032 0)
       (effects (font (size 1.778 1.5113)) (justify left bottom))
     )
-    (property "Footprint" "" (id 2) (at 146.05 130.81 0)
+    (property "Footprint" "oresat0-1u-backplane:1206-C" (id 2) (at 146.05 130.81 0)
       (effects (font (size 1.27 1.27)) hide)
     )
@@
     (pin "2")
   )
-  (symbol (lib_id "oresat0-1u-backplane-eagle-import:FRAME_A_L") (at 17.78 233.68 0) (unit 1)
-    (in_bom yes) (on_board yes)
-    (property "Reference" "#FRAME13" (id 0) (at 17.78 233.68 0)
-      (effects (font (size 1.27 1.27)) hide)
-    )
-    (property "Value" "" (id 1) (at 17.78 233.68 0)
-      (effects (font (size 1.27 1.27)) hide)
-    )
-    (property "Footprint" "" (id 2) (at 17.78 233.68 0)
-      (effects (font (size 1.27 1.27)) hide)
-    )
-    (property "Datasheet" "" (id 3) (at 17.78 233.68 0)
-      (effects (font (size 1.27 1.27)) hide)
-    )
-  )
   (symbol (lib_id "oresat0-1u-backplane-eagle-import:R-US_1206-C") (at 143.51 90.17 0) (unit 1)
     (in_bom yes) (on_board yes)
@@
       (effects (font (size 1.778 1.5113)) (justify left bottom))
     )
-    (property "Value" "" (id 1) (at 144.78 88.392 0)
+    (property "Value" "NP/60.4" (id 1) (at 144.78 88.392 0)
       (effects (font (size 1.778 1.5113)) (justify left bottom))
     )
-    (property "Footprint" "" (id 2) (at 143.51 90.17 0)
+    (property "Footprint" "oresat0-1u-backplane:1206-C" (id 2) (at 143.51 90.17 0)
       (effects (font (size 1.27 1.27)) hide)
     )
@@
   (symbol (lib_id "oresat0-1u-backplane-eagle-import:GND") (at 158.75 146.05 0) (unit 1)
     (in_bom yes) (on_board yes)
-    (property "Reference" "#GND20" (id 0) (at 158.75 146.05 0)
+    (property "Reference" "#GND020" (id 0) (at 158.75 146.05 0)
       (effects (font (size 1.27 1.27)) hide)
     )
-    (property "Value" "" (id 1) (at 158.75 146.05 0)
+    (property "Value" "GND" (id 1) (at 158.75 146.05 0)
       (effects (font (size 1.27 1.27)) hide)
     )
-    (property "Footprint" "" (id 2) (at 158.75 146.05 0)
+    (property "Footprint" "oresat0-1u-backplane:" (id 2) (at 158.75 146.05 0)
       (effects (font (size 1.27 1.27)) hide)
     )
@@
       (effects (font (size 1.778 1.5113)) (justify left bottom))
     )
-    (property "Value" "" (id 1) (at 144.78 98.552 0)
+    (property "Value" "NP/60.4" (id 1) (at 144.78 98.552 0)
       (effects (font (size 1.778 1.5113)) (justify left bottom))
     )
-    (property "Footprint" "" (id 2) (at 143.51 95.25 0)
+    (property "Footprint" "oresat0-1u-backplane:1206-C" (id 2) (at 143.51 95.25 0)
       (effects (font (size 1.27 1.27)) hide)
     )
@@
       (effects (font (size 1.778 1.5113)) (justify left bottom))
     )
-    (property "Value" "" (id 1) (at 147.32 139.192 0)
+    (property "Value" "NP/60.4" (id 1) (at 147.32 139.192 0)
       (effects (font (size 1.778 1.5113)) (justify left bottom))
     )
-    (property "Footprint" "" (id 2) (at 146.05 135.89 0)
+    (property "Footprint" "oresat0-1u-backplane:1206-C" (id 2) (at 146.05 135.89 0)
       (effects (font (size 1.27 1.27)) hide)
     )
@@
       (effects (font (size 1.778 1.5113)) (justify left bottom))
     )
-    (property "Value" "" (id 1) (at 160.274 143.129 0)
+    (property "Value" "1n" (id 1) (at 160.274 143.129 0)
       (effects (font (size 1.778 1.5113)) (justify left bottom))
     )
-    (property "Footprint" "" (id 2) (at 158.75 138.43 0)
+    (property "Footprint" "oresat0-1u-backplane:.0603-C-NOSILK" (id 2) (at 158.75 138.43 0)
       (effects (font (size 1.27 1.27)) hide)
     )
