File: 1u/KiCad/oresat0-1u-backplane/To_-Z_End_Cap.kicad_sch (KiCad schematic)
At the start: 2 parts

Commit message: Fixed DRC errors and warnings
Parts:
- CM8: value (none) -> U.FL-R-SMA; footprint (none) -> oresat0-1u-backplane:U.FL-R-SMT
- J1: value (none) -> 5-104196-5; footprint (none) -> oresat0-1u-backplane:5-104196-5
Changed lines of the file:
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@@
-    )
-  )
-  (symbol (lib_id "oresat0-1u-backplane-eagle-import:FRAME_A_L") (at 190.5 233.68 0) (unit 2)
-    (in_bom yes) (on_board yes)
-    (property "Reference" "#FRAME12" (id 0) (at 190.5 233.68 0)
-      (effects (font (size 1.27 1.27)) hide)
-    )
-    (property "Value" "" (id 1) (at 190.5 233.68 0)
-      (effects (font (size 1.27 1.27)) hide)
-    )
-    (property "Footprint" "" (id 2) (at 190.5 233.68 0)
-      (effects (font (size 1.27 1.27)) hide)
-    )
-    (property "Datasheet" "" (id 3) (at 190.5 233.68 0)
-      (effects (font (size 1.27 1.27)) hide)
-    )
-  )
-  (symbol (lib_id "oresat0-1u-backplane-eagle-import:FRAME_A_L") (at 17.78 233.68 0) (unit 1)
-    (in_bom yes) (on_board yes)
-    (property "Reference" "#FRAME12" (id 0) (at 17.78 233.68 0)
-      (effects (font (size 1.27 1.27)) hide)
-    )
-    (property "Value" "" (id 1) (at 17.78 233.68 0)
-      (effects (font (size 1.27 1.27)) hide)
-    )
-    (property "Footprint" "" (id 2) (at 17.78 233.68 0)
-      (effects (font (size 1.27 1.27)) hide)
-    )
-    (property "Datasheet" "" (id 3) (at 17.78 233.68 0)
-      (effects (font (size 1.27 1.27)) hide)
     )
   )
@@
       (effects (font (size 1.778 1.5113)) (justify left bottom))
     )
-    (property "Value" "" (id 1) (at 109.22 88.9 0)
+    (property "Value" "5-104196-5" (id 1) (at 109.22 88.9 0)
       (effects (font (size 1.778 1.5113)) (justify left bottom))
     )
-    (property "Footprint" "" (id 2) (at 102.87 115.57 0)
+    (property "Footprint" "oresat0-1u-backplane:5-104196-5" (id 2) (at 102.87 115.57 0)
       (effects (font (size 1.27 1.27)) hide)
     )
@@
   (symbol (lib_id "oresat0-1u-backplane-eagle-import:GND") (at 199.39 118.11 0) (unit 1)
     (in_bom yes) (on_board yes)
-    (property "Reference" "#GND8" (id 0) (at 199.39 118.11 0)
+    (property "Reference" "#GND08" (id 0) (at 199.39 118.11 0)
       (effects (font (size 1.27 1.27)) hide)
     )
-    (property "Value" "" (id 1) (at 199.39 118.11 0)
+    (property "Value" "GND" (id 1) (at 199.39 118.11 0)
       (effects (font (size 1.27 1.27)) hide)
     )
-    (property "Footprint" "" (id 2) (at 199.39 118.11 0)
+    (property "Footprint" "oresat0-1u-backplane:" (id 2) (at 199.39 118.11 0)
       (effects (font (size 1.27 1.27)) hide)
     )
@@
       (effects (font (size 1.778 1.5113)) (justify left bottom))
     )
-    (property "Value" "" (id 1) (at 212.09 115.57 0)
+    (property "Value" "U.FL-R-SMA" (id 1) (at 212.09 115.57 0)
       (effects (font (size 1.778 1.5113)) (justify left bottom))
     )
-    (property "Footprint" "" (id 2) (at 205.74 110.49 0)
+    (property "Footprint" "oresat0-1u-backplane:U.FL-R-SMT" (id 2) (at 205.74 110.49 0)
       (effects (font (size 1.27 1.27)) hide)
     )
@@
   (symbol (lib_id "oresat0-1u-backplane-eagle-import:GND") (at 105.41 147.32 0) (unit 1)
     (in_bom yes) (on_board yes)
-    (property "Reference" "#GND6" (id 0) (at 105.41 147.32 0)
+    (property "Reference" "#GND06" (id 0) (at 105.41 147.32 0)
       (effects (font (size 1.27 1.27)) hide)
     )
-    (property "Value" "" (id 1) (at 105.41 147.32 0)
+    (property "Value" "GND" (id 1) (at 105.41 147.32 0)
       (effects (font (size 1.27 1.27)) hide)
     )
-    (property "Footprint" "" (id 2) (at 105.41 147.32 0)
+    (property "Footprint" "oresat0-1u-backplane:" (id 2) (at 105.41 147.32 0)
       (effects (font (size 1.27 1.27)) hide)
     )
