File: oresat-backplane-2u/Slot_18.kicad_sch (KiCad schematic)
At the start: 2 parts

Commit message: Aligned everything to the DXF, should maybe be done I think
Parts:
- CF18.1: footprint oresat-backplane-2u:SFM-110-X1-XXX-D-LC -> oresat-footprints:J-SAMTEC-CF-SFM-110-X1-XXX-D-LC
- CF18.2: footprint oresat-backplane-2u:SFM-120-X1-XXX-D -> oresat-footprints:J-SAMTEC-SFM-120-X1-XXX-D
Changed lines of the file:
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@@
       (effects (font (size 1.27 1.0795)) (justify left bottom))
     )
-    (property "Footprint" "oresat-backplane-2u:SFM-110-X1-XXX-D-LC" (id 2) (at 33.02 66.04 0)
+    (property "Footprint" "oresat-footprints:J-SAMTEC-CF-SFM-110-X1-XXX-D-LC" (id 2) (at 33.02 66.04 0)
       (effects (font (size 1.27 1.27)) hide)
     )
@@
       (effects (font (size 1.27 1.0795)) (justify left bottom))
     )
-    (property "Footprint" "oresat-backplane-2u:SFM-120-X1-XXX-D" (id 2) (at 33.02 157.48 0)
+    (property "Footprint" "oresat-footprints:J-SAMTEC-SFM-120-X1-XXX-D" (id 2) (at 33.02 157.48 0)
       (effects (font (size 1.27 1.27)) hide)
     )
