File: 2U/oresat-0.5/oresat-backplane-2u.kicad_sch (KiCad schematic)
At the start: 0 parts

Commit message: Moved entire schematic to single page
Parts:
- added C1, C12, C13, C14, C15, C16, C17, C18, C19, C2, C20, C3, C4, C5, C6, C7, C8: 10u 25V, Capacitor_SMD:C_1206_3216Metric, symbol Device:C
- added C1.1, C1.2, C20.1, C20.2: 1n, oresat-passives:0603-SMALL, symbol Device:C
- added CF1.2, CF12.2, CF13.2, CF14.2, CF15.2, CF16.2, CF17.2, CF18.2, CF19.2, CF2.2, CF20.2, CF3.2, CF4.2, CF5.2, CF6.2, CF7.2, CF8.2: SFM-120-X1-XXX-D, oresat-connectors:J-SAMTEC-SFM-120-X1-XXX-D, symbol oresat-connectors:J-SAMTEC-TFM-120-01-L-D-RA
- added CF18.1, CF19.1: SFM-110-X1-XXX-D-LC, oresat-connectors:J-SAMTEC-CF-SFM-110-X1-XXX-D-LC, symbol oresat-connectors:J-SAMTEC-TFM-110-01-L-D-RA
- added CM1.1, CM2.1, CM20.1, CM20.2, CM20.3, CM3.2, CM4.2, CM4.3: J-MOLEX-SMPM-73300-0111X, oresat-connectors:J-MOLEX-SMPM-73300-0111X-long, symbol oresat-connectors:J-MOLEX-SMPM-73300-0111X_1
- added J1: m55-6001642, oresat-connectors:m55-6001642, symbol oresat-connectors:m55-6001642
- added R1.1, R1.2, R1.3, R1.4, R20.1, R20.2, R20.3, R20.4: 60.4, Resistor_SMD:R_1206_3216Metric, symbol Device:R_US
- added R20.5, R20.6: 0, oresat-passives:0603-SMALL, symbol Device:R_US
Connections:
- new net: C1.1.1, R1.1.1, R1.2.2
- new net: C20.2.1, R20.3.2, R20.4.1
- new net: C20.1.1, R20.1.2, R20.2.1
- new net: C1.2.1, R1.3.1, R1.4.2
- new net AUX-1: CF18.1.1, CF18.1.2, CF19.1.1, CF19.1.2
- new net AUX-10: CF18.1.19, CF18.1.20, CF19.1.19, CF19.1.20
- new net AUX-2: CF18.1.3, CF18.1.4, CF19.1.3, CF19.1.4
- new net AUX-3: CF18.1.5, CF18.1.6, CF19.1.5, CF19.1.6
- new net AUX-4: CF18.1.7, CF18.1.8, CF19.1.7, CF19.1.8
- new net AUX-5: CF18.1.10, CF18.1.9, CF19.1.10, CF19.1.9
- new net AUX-6: CF18.1.11, CF18.1.12, CF19.1.11, CF19.1.12
- new net AUX-7: CF18.1.13, CF18.1.14, CF19.1.13, CF19.1.14
- new net AUX-8: CF18.1.15, CF18.1.16, CF19.1.15, CF19.1.16
- new net AUX-9: CF18.1.17, CF18.1.18, CF19.1.17, CF19.1.18
- new net C3-UART-RX: CF1.2.38, CF12.2.38, CF13.2.38, CF14.2.38, CF15.2.38, CF16.2.38, CF17.2.38, CF18.2.38, CF19.2.38, CF2.2.38, CF20.2.38, CF3.2.38, CF4.2.38, CF5.2.38, CF6.2.38, CF7.2.38, CF8.2.38, J1.b8 (Pin_b8)
- new net C3-UART-TX: CF1.2.37, CF12.2.37, CF13.2.37, CF14.2.37, CF15.2.37, CF16.2.37, CF17.2.37, CF18.2.37, CF19.2.37, CF2.2.37, CF20.2.37, CF3.2.37, CF4.2.37, CF5.2.37, CF6.2.37, CF7.2.37, CF8.2.37, J1.a7 (Pin_a7)
- new net CAN1_H: CF1.2.33, CF1.2.34, CF12.2.33, CF12.2.34, CF13.2.33, CF13.2.34, CF14.2.33, CF14.2.34, CF15.2.33, CF15.2.34, CF16.2.33, CF16.2.34, CF17.2.33, CF17.2.34, CF18.2.33, CF18.2.34, CF19.2.33, CF19.2.34, CF2.2.33, CF2.2.34, CF20.2.33, CF20.2.34, CF3.2.33, CF3.2.34, CF4.2.33, CF4.2.34, CF5.2.33, CF5.2.34, CF6.2.33, CF6.2.34, CF7.2.33, CF7.2.34, CF8.2.33, CF8.2.34, J1.a6 (Pin_a6), R1.3.2, R20.3.1, R20.5.1
- new net CAN1_L: CF1.2.35, CF1.2.36, CF12.2.35, CF12.2.36, CF13.2.35, CF13.2.36, CF14.2.35, CF14.2.36, CF15.2.35, CF15.2.36, CF16.2.35, CF16.2.36, CF17.2.35, CF17.2.36, CF18.2.35, CF18.2.36, CF19.2.35, CF19.2.36, CF2.2.35, CF2.2.36, CF20.2.35, CF20.2.36, CF3.2.35, CF3.2.36, CF4.2.35, CF4.2.36, CF5.2.35, CF5.2.36, CF6.2.35, CF6.2.36, CF7.2.35, CF7.2.36, CF8.2.35, CF8.2.36, J1.b7 (Pin_b7), R1.4.1, R20.4.2, R20.6.1
- new net CAN2_H: CF1.2.17, CF1.2.18, CF12.2.17, CF12.2.18, CF13.2.17, CF13.2.18, CF14.2.17, CF14.2.18, CF15.2.17, CF15.2.18, CF16.2.17, CF16.2.18, CF17.2.17, CF17.2.18, CF18.2.17, CF18.2.18, CF19.2.17, CF19.2.18, CF2.2.17, CF2.2.18, CF20.2.17, CF20.2.18, CF3.2.17, CF3.2.18, CF4.2.17, CF4.2.18, CF5.2.17, CF5.2.18, CF6.2.17, CF6.2.18, CF7.2.17, CF7.2.18, CF8.2.17, CF8.2.18, J1.a2 (Pin_a2), R1.1.2, R20.1.1, R20.5.2
- new net CAN2_L: CF1.2.19, CF1.2.20, CF12.2.19, CF12.2.20, CF13.2.19, CF13.2.20, CF14.2.19, CF14.2.20, CF15.2.19, CF15.2.20, CF16.2.19, CF16.2.20, CF17.2.19, CF17.2.20, CF18.2.19, CF18.2.20, CF19.2.19, CF19.2.20, CF2.2.19, CF2.2.20, CF20.2.19, CF20.2.20, CF3.2.19, CF3.2.20, CF4.2.19, CF4.2.20, CF5.2.19, CF5.2.20, CF6.2.19, CF6.2.20, CF7.2.19, CF7.2.20, CF8.2.19, CF8.2.20, J1.b3 (Pin_b3), R1.2.1, R20.2.2, R20.6.2
- new net GND: C1.1.2, C1.2, C1.2.2, C12.2, C13.2, C14.2, C15.2, C16.2, C17.2, C18.2, C19.2, C2.2, C20.1.2, C20.2, C20.2.2, C3.2, C4.2, C5.2, C6.2, C7.2, C8.2, CF1.2.27, CF1.2.28, CF1.2.29, CF1.2.30, CF1.2.31, CF1.2.32, CF1.2.LC1, CF1.2.LC2, CF12.2.27, CF12.2.28, CF12.2.29, CF12.2.30, CF12.2.31, CF12.2.32, CF12.2.LC1, CF12.2.LC2, CF13.2.27, CF13.2.28, CF13.2.29, CF13.2.30, CF13.2.31, CF13.2.32, CF13.2.LC1, CF13.2.LC2, CF14.2.27, CF14.2.28, CF14.2.29, CF14.2.30, CF14.2.31, CF14.2.32, CF14.2.LC1, CF14.2.LC2, CF15.2.27, CF15.2.28, CF15.2.29, CF15.2.30, CF15.2.31, CF15.2.32, CF15.2.LC1, CF15.2.LC2, CF16.2.27, CF16.2.28, CF16.2.29, CF16.2.30, CF16.2.31, CF16.2.32, CF16.2.LC1, CF16.2.LC2, CF17.2.27, CF17.2.28, CF17.2.29, CF17.2.30, CF17.2.31, CF17.2.32, CF17.2.LC1, CF17.2.LC2, CF18.1.LC1, CF18.1.LC2, CF18.2.27, CF18.2.28, CF18.2.29, CF18.2.30, CF18.2.31, CF18.2.32, CF18.2.LC1, CF18.2.LC2, CF19.1.LC1, CF19.1.LC2, CF19.2.27, CF19.2.28, CF19.2.29, CF19.2.30, CF19.2.31, CF19.2.32, CF19.2.LC1, CF19.2.LC2, CF2.2.27, CF2.2.28, CF2.2.29, CF2.2.30, CF2.2.31, CF2.2.32, CF2.2.LC1, CF2.2.LC2, CF20.2.27, CF20.2.28, CF20.2.29, CF20.2.30, CF20.2.31, CF20.2.32, CF20.2.LC1, CF20.2.LC2, CF3.2.27, CF3.2.28, CF3.2.29, CF3.2.30, CF3.2.31, CF3.2.32, CF3.2.LC1, CF3.2.LC2, CF4.2.27, CF4.2.28, CF4.2.29, CF4.2.30, CF4.2.31, CF4.2.32, CF4.2.LC1, CF4.2.LC2, CF5.2.27, CF5.2.28, CF5.2.29, CF5.2.30, CF5.2.31, CF5.2.32, CF5.2.LC1, CF5.2.LC2, CF6.2.27, CF6.2.28, CF6.2.29, CF6.2.30, CF6.2.31, CF6.2.32, CF6.2.LC1, CF6.2.LC2, CF7.2.27, CF7.2.28, CF7.2.29, CF7.2.30, CF7.2.31, CF7.2.32, CF7.2.LC1, CF7.2.LC2, CF8.2.27, CF8.2.28, CF8.2.29, CF8.2.30, CF8.2.31, CF8.2.32, CF8.2.LC1, CF8.2.LC2, CM1.1.GND (SHIELD1), CM2.1.GND (SHIELD1), CM20.1.GND (SHIELD1), CM20.2.GND (SHIELD1), CM20.3.GND (SHIELD1), CM3.2.GND (SHIELD1), CM4.2.GND (SHIELD1), CM4.3.GND (SHIELD1), J1.b4 (Pin_b4), J1.b5 (Pin_b5), J1.b6 (Pin_b6), J1.mech
- new net HELICAL-DEPLOY: CF1.2.7, CF1.2.8, CF12.2.7, CF12.2.8, CF13.2.7, CF13.2.8, CF14.2.7, CF14.2.8, CF15.2.7, CF15.2.8, CF16.2.7, CF16.2.8, CF17.2.7, CF17.2.8, CF18.2.7, CF18.2.8, CF19.2.7, CF19.2.8, CF2.2.7, CF2.2.8, CF20.2.7, CF20.2.8, CF3.2.7, CF3.2.8, CF4.2.7, CF4.2.8, CF5.2.7, CF5.2.8, CF6.2.7, CF6.2.8, CF7.2.7, CF7.2.8, CF8.2.7, CF8.2.8
- new net L-ANT: CM20.2.RF-DOWN (RF), CM4.2.RF-DOWN (RF)
- new net L1-ANT: CM20.1.RF-DOWN (RF), CM3.2.RF-DOWN (RF)
- new net MAG-POWER: CF1.2.5, CF1.2.6, CF12.2.5, CF12.2.6, CF13.2.5, CF13.2.6, CF14.2.5, CF14.2.6, CF15.2.5, CF15.2.6, CF16.2.5, CF16.2.6, CF17.2.5, CF17.2.6, CF18.2.5, CF18.2.6, CF19.2.5, CF19.2.6, CF2.2.5, CF2.2.6, CF20.2.5, CF20.2.6, CF3.2.5, CF3.2.6, CF4.2.5, CF4.2.6, CF5.2.5, CF5.2.6, CF6.2.5, CF6.2.6, CF7.2.5, CF7.2.6, CF8.2.5, CF8.2.6
- new net MAG-SCL: CF1.2.3, CF1.2.4, CF12.2.3, CF12.2.4, CF13.2.3, CF13.2.4, CF14.2.3, CF14.2.4, CF15.2.3, CF15.2.4, CF16.2.3, CF16.2.4, CF17.2.3, CF17.2.4, CF18.2.3, CF18.2.4, CF19.2.3, CF19.2.4, CF2.2.3, CF2.2.4, CF20.2.3, CF20.2.4, CF3.2.3, CF3.2.4, CF4.2.3, CF4.2.4, CF5.2.3, CF5.2.4, CF6.2.3, CF6.2.4, CF7.2.3, CF7.2.4, CF8.2.3, CF8.2.4
- new net MAG-SDA: CF1.2.1, CF1.2.2, CF12.2.1, CF12.2.2, CF13.2.1, CF13.2.2, CF14.2.1, CF14.2.2, CF15.2.1, CF15.2.2, CF16.2.1, CF16.2.2, CF17.2.1, CF17.2.2, CF18.2.1, CF18.2.2, CF19.2.1, CF19.2.2, CF2.2.1, CF2.2.2, CF20.2.1, CF20.2.2, CF3.2.1, CF3.2.2, CF4.2.1, CF4.2.2, CF5.2.1, CF5.2.2, CF6.2.1, CF6.2.2, CF7.2.1, CF7.2.2, CF8.2.1, CF8.2.2
- new net OPD_PWR: CF1.2.15, CF1.2.16, CF12.2.15, CF12.2.16, CF13.2.15, CF13.2.16, CF14.2.15, CF14.2.16, CF15.2.15, CF15.2.16, CF16.2.15, CF16.2.16, CF17.2.15, CF17.2.16, CF18.2.15, CF18.2.16, CF19.2.15, CF19.2.16, CF2.2.15, CF2.2.16, CF20.2.15, CF20.2.16, CF3.2.15, CF3.2.16, CF4.2.15, CF4.2.16, CF5.2.15, CF5.2.16, CF6.2.15, CF6.2.16, CF7.2.15, CF7.2.16, CF8.2.15, CF8.2.16, J1.b2 (Pin_b2)
- new net OPD_SCL: CF1.2.13, CF1.2.14, CF12.2.13, CF12.2.14, CF13.2.13, CF13.2.14, CF14.2.13, CF14.2.14, CF15.2.13, CF15.2.14, CF16.2.13, CF16.2.14, CF17.2.13, CF17.2.14, CF18.2.13, CF18.2.14, CF19.2.13, CF19.2.14, CF2.2.13, CF2.2.14, CF20.2.13, CF20.2.14, CF3.2.13, CF3.2.14, CF4.2.13, CF4.2.14, CF5.2.13, CF5.2.14, CF6.2.13, CF6.2.14, CF7.2.13, CF7.2.14, CF8.2.13, CF8.2.14, J1.a1 (Pin_a1)
- new net OPD_SDA: CF1.2.11, CF1.2.12, CF12.2.11, CF12.2.12, CF13.2.11, CF13.2.12, CF14.2.11, CF14.2.12, CF15.2.11, CF15.2.12, CF16.2.11, CF16.2.12, CF17.2.11, CF17.2.12, CF18.2.11, CF18.2.12, CF19.2.11, CF19.2.12, CF2.2.11, CF2.2.12, CF20.2.11, CF20.2.12, CF3.2.11, CF3.2.12, CF4.2.11, CF4.2.12, CF5.2.11, CF5.2.12, CF6.2.11, CF6.2.12, CF7.2.11, CF7.2.12, CF8.2.11, CF8.2.12, J1.b1 (Pin_b1)
- new net S-ANT: CM1.1.RF-DOWN (RF), CM2.1.RF-DOWN (RF)
- new net TURNSTILE-DEPLOY: CF1.2.10, CF1.2.9, CF12.2.10, CF12.2.9, CF13.2.10, CF13.2.9, CF14.2.10, CF14.2.9, CF15.2.10, CF15.2.9, CF16.2.10, CF16.2.9, CF17.2.10, CF17.2.9, CF18.2.10, CF18.2.9, CF19.2.10, CF19.2.9, CF2.2.10, CF2.2.9, CF20.2.10, CF20.2.9, CF3.2.10, CF3.2.9, CF4.2.10, CF4.2.9, CF5.2.10, CF5.2.9, CF6.2.10, CF6.2.9, CF7.2.10, CF7.2.9, CF8.2.10, CF8.2.9
- new net UHF-ANT: CM20.3.RF-DOWN (RF), CM4.3.RF-DOWN (RF)
- new net VBUS: C1.1, C12.1, C13.1, C14.1, C15.1, C16.1, C17.1, C18.1, C19.1, C2.1, C20.1, C3.1, C4.1, C5.1, C6.1, C7.1, C8.1, CF1.2.21, CF1.2.22, CF1.2.23, CF1.2.24, CF1.2.25, CF1.2.26, CF12.2.21, CF12.2.22, CF12.2.23, CF12.2.24, CF12.2.25, CF12.2.26, CF13.2.21, CF13.2.22, CF13.2.23, CF13.2.24, CF13.2.25, CF13.2.26, CF14.2.21, CF14.2.22, CF14.2.23, CF14.2.24, CF14.2.25, CF14.2.26, CF15.2.21, CF15.2.22, CF15.2.23, CF15.2.24, CF15.2.25, CF15.2.26, CF16.2.21, CF16.2.22, CF16.2.23, CF16.2.24, CF16.2.25, CF16.2.26, CF17.2.21, CF17.2.22, CF17.2.23, CF17.2.24, CF17.2.25, CF17.2.26, CF18.2.21, CF18.2.22, CF18.2.23, CF18.2.24, CF18.2.25, CF18.2.26, CF19.2.21, CF19.2.22, CF19.2.23, CF19.2.24, CF19.2.25, CF19.2.26, CF2.2.21, CF2.2.22, CF2.2.23, CF2.2.24, CF2.2.25, CF2.2.26, CF20.2.21, CF20.2.22, CF20.2.23, CF20.2.24, CF20.2.25, CF20.2.26, CF3.2.21, CF3.2.22, CF3.2.23, CF3.2.24, CF3.2.25, CF3.2.26, CF4.2.21, CF4.2.22, CF4.2.23, CF4.2.24, CF4.2.25, CF4.2.26, CF5.2.21, CF5.2.22, CF5.2.23, CF5.2.24, CF5.2.25, CF5.2.26, CF6.2.21, CF6.2.22, CF6.2.23, CF6.2.24, CF6.2.25, CF6.2.26, CF7.2.21, CF7.2.22, CF7.2.23, CF7.2.24, CF7.2.25, CF7.2.26, CF8.2.21, CF8.2.22, CF8.2.23, CF8.2.24, CF8.2.25, CF8.2.26, J1.a3 (Pin_a3), J1.a4 (Pin_a4), J1.a5 (Pin_a5)
- new net ~{SD}: CF1.2.39, CF1.2.40, CF12.2.39, CF12.2.40, CF13.2.39, CF13.2.40, CF14.2.39, CF14.2.40, CF15.2.39, CF15.2.40, CF16.2.39, CF16.2.40, CF17.2.39, CF17.2.40, CF18.2.39, CF18.2.40, CF19.2.39, CF19.2.40, CF2.2.39, CF2.2.40, CF20.2.39, CF20.2.40, CF3.2.39, CF3.2.40, CF4.2.39, CF4.2.40, CF5.2.39, CF5.2.40, CF6.2.39, CF6.2.40, CF7.2.39, CF7.2.40, CF8.2.39, CF8.2.40, J1.a8 (Pin_a8)
Other:
- removed sheet Slot 1
- removed sheet Slot 10
- removed sheet Slot 11
- removed sheet Slot 12
- removed sheet Slot 13
- removed sheet Slot 14
- removed sheet Slot 15
- removed sheet Slot 16
- removed sheet Slot 17
- removed sheet Slot 18
- removed sheet Slot 19
- removed sheet Slot 2
- removed sheet Slot 20
- removed sheet Slot 3
- removed sheet Slot 4
- removed sheet Slot 5
- removed sheet Slot 6
- removed sheet Slot 7
- removed sheet Slot 8
- removed sheet Slot 9
- note added: "Use R20.5,R20.6 to bridge CAN1 and CAN2"

Commit message: Ready for fab I think
Other:
- note added: "Aux connectors"
- note added: "Debug Connector"
- moved on the sheet: CF18.1, CF19.1, J1, R20.5, R20.6

Commit message: Fixed backplane connector library names
Parts:
- CF1.2, CF12.2, CF13.2, CF14.2, CF15.2, CF16.2, CF17.2, CF18.2, CF19.2, CF2.2, CF20.2, CF3.2, CF4.2, CF5.2, CF6.2, CF7.2, CF8.2: symbol oresat-connectors:J-SAMTEC-TFM-120-01-L-D-RA -> oresat-connectors:J-SAMTEC-SFM-120-X1-XXX-D
Changed lines of the file:
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@@
     )
   )
-  (symbol (lib_id "oresat-connectors:J-SAMTEC-TFM-120-01-L-D-RA") (at 283.21 186.69 0) (unit 1)
+  (symbol (lib_id "oresat-connectors:J-SAMTEC-SFM-120-X1-XXX-D") (at 283.21 186.69 0) (unit 1)
     (in_bom yes) (on_board yes)
     (property "Reference" "CF19.2" (id 0) (at 280.67 134.62 0)
@@
     (pin "2")
   )
-  (symbol (lib_id "oresat-connectors:J-SAMTEC-TFM-120-01-L-D-RA") (at 172.72 186.69 0) (unit 1)
+  (symbol (lib_id "oresat-connectors:J-SAMTEC-SFM-120-X1-XXX-D") (at 172.72 186.69 0) (unit 1)
     (in_bom yes) (on_board yes)
     (property "Reference" "CF16.2" (id 0) (at 170.18 134.62 0)
@@
     (pin "2")
   )
-  (symbol (lib_id "oresat-connectors:J-SAMTEC-TFM-120-01-L-D-RA") (at 320.04 67.31 0) (unit 1)
+  (symbol (lib_id "oresat-connectors:J-SAMTEC-SFM-120-X1-XXX-D") (at 320.04 67.31 0) (unit 1)
     (in_bom yes) (on_board yes)
     (property "Reference" "CF8.2" (id 0) (at 317.5 15.24 0)
@@
     (pin "1")
   )
-  (symbol (lib_id "oresat-connectors:J-SAMTEC-TFM-120-01-L-D-RA") (at 25.4 186.69 0) (unit 1)
+  (symbol (lib_id "oresat-connectors:J-SAMTEC-SFM-120-X1-XXX-D") (at 25.4 186.69 0) (unit 1)
     (in_bom yes) (on_board yes)
     (property "Reference" "CF12.2" (id 0) (at 22.86 134.62 0)
@@
     (pin "1")
   )
-  (symbol (lib_id "oresat-connectors:J-SAMTEC-TFM-120-01-L-D-RA") (at 209.55 67.31 0) (unit 1)
+  (symbol (lib_id "oresat-connectors:J-SAMTEC-SFM-120-X1-XXX-D") (at 209.55 67.31 0) (unit 1)
     (in_bom yes) (on_board yes)
     (property "Reference" "CF5.2" (id 0) (at 207.01 15.24 0)
@@
     (pin "1")
   )
-  (symbol (lib_id "oresat-connectors:J-SAMTEC-TFM-120-01-L-D-RA") (at 135.89 67.31 0) (unit 1)
+  (symbol (lib_id "oresat-connectors:J-SAMTEC-SFM-120-X1-XXX-D") (at 135.89 67.31 0) (unit 1)
     (in_bom yes) (on_board yes)
     (property "Reference" "CF3.2" (id 0) (at 133.35 15.24 0)
@@
     (pin "mech")
   )
-  (symbol (lib_id "oresat-connectors:J-SAMTEC-TFM-120-01-L-D-RA") (at 25.4 68.58 0) (unit 1)
+  (symbol (lib_id "oresat-connectors:J-SAMTEC-SFM-120-X1-XXX-D") (at 25.4 68.58 0) (unit 1)
     (in_bom yes) (on_board yes)
     (property "Reference" "CF1.2" (id 0) (at 22.86 16.51 0)
@@
     (pin "LC2")
   )
-  (symbol (lib_id "oresat-connectors:J-SAMTEC-TFM-120-01-L-D-RA") (at 99.06 67.31 0) (unit 1)
+  (symbol (lib_id "oresat-connectors:J-SAMTEC-SFM-120-X1-XXX-D") (at 99.06 67.31 0) (unit 1)
     (in_bom yes) (on_board yes)
     (property "Reference" "CF2.2" (id 0) (at 96.52 15.24 0)
@@
     (pin "1")
   )
-  (symbol (lib_id "oresat-connectors:J-SAMTEC-TFM-120-01-L-D-RA") (at 99.06 186.69 0) (unit 1)
+  (symbol (lib_id "oresat-connectors:J-SAMTEC-SFM-120-X1-XXX-D") (at 99.06 186.69 0) (unit 1)
     (in_bom yes) (on_board yes)
     (property "Reference" "CF14.2" (id 0) (at 96.52 134.62 0)
@@
     (pin "LC2")
   )
-  (symbol (lib_id "oresat-connectors:J-SAMTEC-TFM-120-01-L-D-RA") (at 283.21 67.31 0) (unit 1)
+  (symbol (lib_id "oresat-connectors:J-SAMTEC-SFM-120-X1-XXX-D") (at 283.21 67.31 0) (unit 1)
     (in_bom yes) (on_board yes)
     (property "Reference" "CF7.2" (id 0) (at 280.67 15.24 0)
@@
     (pin "1")
   )
-  (symbol (lib_id "oresat-connectors:J-SAMTEC-TFM-120-01-L-D-RA") (at 246.38 186.69 0) (unit 1)
+  (symbol (lib_id "oresat-connectors:J-SAMTEC-SFM-120-X1-XXX-D") (at 246.38 186.69 0) (unit 1)
     (in_bom yes) (on_board yes)
     (property "Reference" "CF18.2" (id 0) (at 243.84 134.62 0)
@@
     (pin "2")
   )
-  (symbol (lib_id "oresat-connectors:J-SAMTEC-TFM-120-01-L-D-RA") (at 172.72 67.31 0) (unit 1)
+  (symbol (lib_id "oresat-connectors:J-SAMTEC-SFM-120-X1-XXX-D") (at 172.72 67.31 0) (unit 1)
     (in_bom yes) (on_board yes)
     (property "Reference" "CF4.2" (id 0) (at 170.18 15.24 0)
@@
     (pin "1")
   )
-  (symbol (lib_id "oresat-connectors:J-SAMTEC-TFM-120-01-L-D-RA") (at 209.55 186.69 0) (unit 1)
+  (symbol (lib_id "oresat-connectors:J-SAMTEC-SFM-120-X1-XXX-D") (at 209.55 186.69 0) (unit 1)
     (in_bom yes) (on_board yes)
     (property "Reference" "CF17.2" (id 0) (at 207.01 134.62 0)
@@
     (pin "1")
   )
-  (symbol (lib_id "oresat-connectors:J-SAMTEC-TFM-120-01-L-D-RA") (at 62.23 186.69 0) (unit 1)
+  (symbol (lib_id "oresat-connectors:J-SAMTEC-SFM-120-X1-XXX-D") (at 62.23 186.69 0) (unit 1)
     (in_bom yes) (on_board yes)
     (property "Reference" "CF13.2" (id 0) (at 59.69 134.62 0)
@@
     (pin "LC2")
   )
-  (symbol (lib_id "oresat-connectors:J-SAMTEC-TFM-120-01-L-D-RA") (at 320.04 186.69 0) (unit 1)
+  (symbol (lib_id "oresat-connectors:J-SAMTEC-SFM-120-X1-XXX-D") (at 320.04 186.69 0) (unit 1)
     (in_bom yes) (on_board yes)
     (property "Reference" "CF20.2" (id 0) (at 317.5 134.62 0)
@@
     (pin "2")
   )
-  (symbol (lib_id "oresat-connectors:J-SAMTEC-TFM-120-01-L-D-RA") (at 135.89 186.69 0) (unit 1)
+  (symbol (lib_id "oresat-connectors:J-SAMTEC-SFM-120-X1-XXX-D") (at 135.89 186.69 0) (unit 1)
     (in_bom yes) (on_board yes)
     (property "Reference" "CF15.2" (id 0) (at 133.35 134.62 0)
@@
     (pin "2")
   )
-  (symbol (lib_id "oresat-connectors:J-SAMTEC-TFM-120-01-L-D-RA") (at 246.38 67.31 0) (unit 1)
+  (symbol (lib_id "oresat-connectors:J-SAMTEC-SFM-120-X1-XXX-D") (at 246.38 67.31 0) (unit 1)
     (in_bom yes) (on_board yes)
     (property "Reference" "CF6.2" (id 0) (at 243.84 15.24 0)
