File: 3U/oresat-backplane-3u/3U backplane.kicad_sch (KiCad schematic)
At the start: 81 parts, among them J1 m55-6001642

Commit message: Rough draft
Lots more cleaning up to be done
Parts:
- removed CF28.1, CF29.1: SFM-110-X1-XXX-D-LC, oresat-connectors:J-SAMTEC-CF-SFM-110-X1-XXX-D-LC, symbol oresat-connectors:J-SAMTEC-TFM-110-01-L-D-RA
Other:
- moved on the sheet: CM1.1, CM1.2, CM1.3, CM12.1, CM12.2, CM3.2, CM3.3, CM4.2, J1
