File: 3U/oresat-backplane-3u/3U backplane.kicad_pcb (KiCad board)
At the start: 4 copper layers, 77 parts, among them J1 m55-6001642

Commit message: Rough draft
Lots more cleaning up to be done
Parts:
- removed CF28.1, CF29.1: SFM-110-X1-XXX-D-LC, oresat-connectors:J-SAMTEC-CF-SFM-110-X1-XXX-D-LC
- J1: moved to B.Cu
- moved J1 2.67 mm to (118.2, -21.5)
- moved CF12.1 0.11 mm to (128.9, 48.3)
Routing:
- net VBUS: track 8.51 -> 78.8 mm, vias 0 -> 3
- net OPD_SCL: track 344.3 -> 388.0 mm, vias 0 -> 1
- net OPD_SDA: track 344.5 -> 385.9 mm, vias 0 -> 1
- net CAN2_H: track 353.0 -> 394.1 mm, vias 0 -> 1
- net OPD_PWR: track 344.2 -> 383.0 mm, vias 0 -> 1
- net CAN2_L: track 353.5 -> 389.9 mm, vias 0 -> 1
- net CAN1_H: track 353.1 -> 384.1 mm, vias 0 -> 1
- net C3-UART-TX: track 347.7 -> 375.3 mm, vias 0 -> 1
- net CAN1_L: track 354.9 -> 380.3 mm, vias 0 -> 1
- net ~{SD}: track 367.3 -> 391.8 mm, vias 0 -> 2
- net C3-UART-RX: track 351.1 -> 374.0 mm, vias 0 -> 1
- net AUX-9: track 11.3 -> 0.00 mm
- net AUX-8: track 11.3 -> 0.00 mm
- net AUX-7: track 11.3 -> 0.00 mm
- net AUX-6: track 11.3 -> 0.00 mm
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Other:
- board text added: "1"
- board text added: "10"
- board text added: "11"
- board text added: "12"
- board text added: "13"
- board text added: "14"
- board text added: "15"
- board text added: "16"
- board text added: "2"
- board text added: "2025-09-30"
- board text added: "3"
- board text added: "4"
- board text added: "5"
- board text added: "6"
- board text added: "7"
- board text added: "8"
- board text added: "9"
- board text added: "A"
- board text added: "A0"
- board text added: "B"
- board text added: "D"
- board text added: "E"
- board text added: "F"
- board text added: "FIRST ANGLE PROJECTION"
- board text added: "G"
- board text added: "H"
- board text added: "I"
- board text added: "J"
- board text added: "K"
- board text added: "L"
- board text added: "SAVANNAH KRUPA"
- board text added: "SIGNATURE"
- board text added: "UNLESS OTHERWISE SPECIFIED, DIMENSIONS ARE IN MILLIMETERS"
- board text removed: "10/04/2025"
- board text removed: "JACOB LUTZ"
- board text removed: "Potato"
- board text removed: "THIRD ANGLE PROJECTION"
- board text removed: "UNLESS OTHERWISE SPECIFIED, DIMENSIONS ARE IN INCHES"

Commit message: Most up to date
Parts:
- added CF19.1: SFM-110-X1-XXX-D-LC, oresat-footprints:J-SAMTEC-CF-SFM-110-X1-XXX-D-LC, F.Cu at (122.5, 5.08)
- added CF19.1: SFM-110-X1-XXX-D-LC, oresat-footprints:J-SAMTEC-CF-SFM-110-X1-XXX-D-LC, F.Cu at (122.5, 191.0)
- added CF19.1: SFM-110-X1-XXX-D-LC, oresat-footprints:J-SAMTEC-CF-SFM-110-X1-XXX-D-LC, F.Cu at (122.5, 107.7)
- added CF19.1: SFM-110-X1-XXX-D-LC, oresat-footprints:J-SAMTEC-CF-SFM-110-X1-XXX-D-LC, F.Cu at (122.5, 15.1)
- added CF19.1: SFM-110-X1-XXX-D-LC, oresat-footprints:J-SAMTEC-CF-SFM-110-X1-XXX-D-LC, F.Cu at (122.5, -4.92)
- added CF19.1: SFM-110-X1-XXX-D-LC, oresat-footprints:J-SAMTEC-CF-SFM-110-X1-XXX-D-LC, F.Cu at (122.5, 151.0)
- added CF19.1: SFM-110-X1-XXX-D-LC, oresat-footprints:J-SAMTEC-CF-SFM-110-X1-XXX-D-LC, F.Cu at (122.5, 181.0)
- added CF19.1: SFM-110-X1-XXX-D-LC, oresat-footprints:J-SAMTEC-CF-SFM-110-X1-XXX-D-LC, F.Cu at (122.5, 97.8)
- added CF19.1: SFM-110-X1-XXX-D-LC, oresat-footprints:J-SAMTEC-CF-SFM-110-X1-XXX-D-LC, F.Cu at (122.5, -54.9)
- added CF19.1: SFM-110-X1-XXX-D-LC, oresat-footprints:J-SAMTEC-CF-SFM-110-X1-XXX-D-LC, F.Cu at (122.5, 35.1)
- added CF19.1: SFM-110-X1-XXX-D-LC, oresat-footprints:J-SAMTEC-CF-SFM-110-X1-XXX-D-LC, F.Cu at (122.5, 210.9)
- added CF19.1: SFM-110-X1-XXX-D-LC, oresat-footprints:J-SAMTEC-CF-SFM-110-X1-XXX-D-LC, F.Cu at (122.5, 231.0)
- added CF19.1: SFM-110-X1-XXX-D-LC, oresat-footprints:J-SAMTEC-CF-SFM-110-X1-XXX-D-LC, F.Cu at (122.5, 201.0)
- added CF19.1: SFM-110-X1-XXX-D-LC, oresat-footprints:J-SAMTEC-CF-SFM-110-X1-XXX-D-LC, F.Cu at (122.5, 25.0)
- added CF19.1: SFM-110-X1-XXX-D-LC, oresat-footprints:J-SAMTEC-CF-SFM-110-X1-XXX-D-LC, F.Cu at (122.5, 58.3)
- added CF19.1: SFM-110-X1-XXX-D-LC, oresat-footprints:J-SAMTEC-CF-SFM-110-X1-XXX-D-LC, F.Cu at (122.5, 117.7)
- added CF19.1: SFM-110-X1-XXX-D-LC, oresat-footprints:J-SAMTEC-CF-SFM-110-X1-XXX-D-LC, F.Cu at (122.5, -44.9)
- added CF19.1: SFM-110-X1-XXX-D-LC, oresat-footprints:J-SAMTEC-CF-SFM-110-X1-XXX-D-LC, F.Cu at (122.5, 141.0)
- added CF19.1: SFM-110-X1-XXX-D-LC, oresat-footprints:J-SAMTEC-CF-SFM-110-X1-XXX-D-LC, F.Cu at (122.5, -34.9)
- added CF19.1: SFM-110-X1-XXX-D-LC, oresat-footprints:J-SAMTEC-CF-SFM-110-X1-XXX-D-LC, F.Cu at (122.5, 170.9)
- added CF19.1: SFM-110-X1-XXX-D-LC, oresat-footprints:J-SAMTEC-CF-SFM-110-X1-XXX-D-LC, F.Cu at (122.5, -14.9)
- added CF19.1: SFM-110-X1-XXX-D-LC, oresat-footprints:J-SAMTEC-CF-SFM-110-X1-XXX-D-LC, F.Cu at (122.5, -24.9)
- added CF19.1: SFM-110-X1-XXX-D-LC, oresat-footprints:J-SAMTEC-CF-SFM-110-X1-XXX-D-LC, F.Cu at (122.5, 161.0)
- added CF19.1: SFM-110-X1-XXX-D-LC, oresat-footprints:J-SAMTEC-CF-SFM-110-X1-XXX-D-LC, F.Cu at (122.5, 221.0)
Routing:
- net TURNSTILE-DEPLOY: track 343.0 -> 344.6 mm
- net HELICAL-DEPLOY: track 343.1 -> 344.4 mm
- net OPD_SCL: track 388.0 -> 389.2 mm
- net OPD_PWR: track 383.0 -> 384.1 mm
- net OPD_SDA: track 385.9 -> 386.6 mm
