File: 3U/oresat-backplane-3u-esi/oresat-backplane-3u-sch-rf.kicad_sch (KiCad schematic)
At the start: 1 part

Commit message: Cleaned up the files Shae was trying to clean up
Parts:
- removed CM1.3: J-MOLEX-SMPM-73300-0111X, oresat-connectors:J-MOLEX-SMPM-73300-0111X-long, symbol oresat-connectors:J-MOLEX-SMPM-73300-0111X_1
- added CM.3.3, CM1.1, CM1.11, CM1.30, CM2.4, CM3.30: 0733000110, oresat-connectors:J-MOLEX-SMPM-73300-0111X-long, symbol oresat-connectors:J-MOLEX-SMPM-73300-0111X_1
Connections:
- net GND: now also CM.3.3.GND (SHIELD1), CM1.1.GND (SHIELD1), CM1.11.GND (SHIELD1), CM1.30.GND (SHIELD1), CM2.4.GND (SHIELD1), CM3.30.GND (SHIELD1)
- new net GPS-L1: CM1.30.RF-DOWN (RF), CM2.4.RF-DOWN (RF)
- new net S-BAND: CM1.1.RF-DOWN (RF), CM1.11.RF-DOWN (RF)
- new net UHF: CM.3.3.RF-DOWN (RF), CM3.30.RF-DOWN (RF)
Other:
- company: Portland State Aerospace Society -> PSAS / ESI
- title: Generic OreSat 3U Backplane -> OreSat 3U Backplane for ESI
